File: proto_II/proto_II_kicad/assembly/proto_II_assembly.kicad_pcb (KiCad board)
At the start: 2 copper layers, 100 x 97 mm, 107 parts, among them J1 BOOT_CFG, J2 SNSR_I2C, J3 SNSR_PWR, J4 Vin, J5 RS485_A, J6 RS485_B, J7 ISO_GND, J8 SWD_DBG, SW1 RST, SW2 MODBUS_ADDR, SW3 USR_BTN, U1 STM32F103C8Tx, U2 TPS54331, U3 XC6206P332MR, U4 ADM2587E, Y1 HSE, Y2 LSE

Commit message: tmp: more fixes
Parts:
- added C11: 30p, Capacitor_SMD:C_0603_1608Metric_Pad1.05x0.95mm_HandSolder, F.Cu at (110.4, 20.3)
- added C12: 30p, Capacitor_SMD:C_0603_1608Metric_Pad1.05x0.95mm_HandSolder, F.Cu at (114.8, 20.3)
- added R3: 560, Resistor_SMD:R_0603_1608Metric_Pad1.05x0.95mm_HandSolder, F.Cu at (119.1, 20.3)
- C16: renamed from C14; footprint Capacitor_SMD:CP_Elec_6.3x5.7 -> Capacitor_SMD:C_1206_3216Metric_Pad1.42x1.75mm_HandSolder
- C17: renamed from C15; footprint Capacitor_SMD:CP_Elec_6.3x5.7 -> Capacitor_SMD:C_1206_3216Metric_Pad1.42x1.75mm_HandSolder
- C23: renamed from C21; value 47u -> 10u; footprint Capacitor_SMD:CP_Elec_6.3x5.7 -> Capacitor_SMD:C_1206_3216Metric_Pad1.42x1.75mm_HandSolder
- C24: renamed from C22; value 47u -> 10u; footprint Capacitor_SMD:CP_Elec_6.3x5.7 -> Capacitor_SMD:C_1206_3216Metric_Pad1.42x1.75mm_HandSolder
- C28: renamed from C26; footprint Capacitor_SMD:CP_Elec_6.3x5.7 -> Capacitor_SMD:C_1206_3216Metric_Pad1.42x1.75mm_HandSolder
- C33: renamed from C31; footprint Capacitor_SMD:CP_Elec_6.3x5.7 -> Capacitor_SMD:C_1206_3216Metric_Pad1.42x1.75mm_HandSolder
- D1: value PWR_LED -> BLUE_LED
- D2: value USR1_LED -> BLUE_LED
- D3: value USR2_LED -> BLUE_LED
- D4: value DI_LED -> BLUE_LED
- D5: value RO_LED -> BLUE_LED
- Y1: footprint Project:Murata_CSTCE8M0V53-R0-3Pin_3.2x1.1mm_HandSoldering -> Crystal:Crystal_SMD_5032-2Pin_5.0x3.2mm_HandSoldering
- moved Y1 76.9 mm to (113.4, 16.7)
- renumbered C11 to C13, C12 to C14, C13 to C15, C16 to C18, C17 to C19, C18 to C20, C19 to C21, C20 to C22, C23 to C25, C24 to C26, C25 to C27, C27 to C29, C28 to C30, C29 to C31, C30 to C32, C32 to C34, C33 to C35, R9 to R10, R10 to R11, R11 to R12, R12 to R13, R13 to R14, R14 to R15, R15 to R16, R16 to R17, R17 to R18, R18 to R19, R19 to R20, R20 to R21, R21 to R22, R22 to R23, R23 to R24, R3 to R4, R4 to R5, R5 to R6, R6 to R7, R7 to R8, R8 to R9
Connections:
- Y1 pad 1: /OSC_IN -> Net-(C11-Pad1)
- Y1 pad 2: GND -> /OSC_IN
Routing:
- net +5VD: track 45.6 -> 0.00 mm
- net /UART3_TX: track 182.2 -> 160.7 mm, vias 6 -> 4
- net /rs485/DE_XMTR: track 14.7 -> 0.00 mm
- net /DE~RE: track 101.7 -> 89.3 mm
- net /rs485/RE_XMTR: track 12.2 -> 0.00 mm
- net /RS485_B: track 30.1 -> 19.2 mm
- net /RS485_A: track 17.5 -> 8.77 mm
- net /UART3_RX: track 166.4 -> 157.8 mm
- net /rs485/DI_XMTR: track 6.82 -> 0.00 mm
- net /rs485/RO_XMTR: track 6.80 -> 0.00 mm
- net GND: track 116.3 -> 110.6 mm, vias 148 -> 147
- net GNDD: track 7.00 -> 1.98 mm, vias 38 -> 34
- net /OSC_OUT: track 4.85 -> 0.00 mm
- net +5V: track 143.6 -> 139.4 mm
- net /OSC_IN: track 5.11 -> 1.09 mm
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
Commit message: tmp: layout started
Parts:
- removed J1: BOOT_CFG, Connector_PinHeader_2.54mm:PinHeader_2x04_P2.54mm_Vertical_SMD
- added C36: 10n, Capacitor_SMD:C_1206_3216Metric_Pad1.42x1.75mm_HandSolder, F.Cu at (75.7, 104.9)
- added JP2: JP, Button_Switch_SMD:SW_DIP_SPSTx01_Slide_9.78x4.72mm_W8.61mm_P2.54mm, F.Cu at (101.4, 112.5)
- added L2: FB, Inductor_SMD:L_0805_2012Metric_Pad1.15x1.40mm_HandSolder, F.Cu at (66.1, 109.2)
- added L3: FB, Inductor_SMD:L_0805_2012Metric_Pad1.15x1.40mm_HandSolder, F.Cu at (66.1, 107.1)
- D6: footprint Diode_SMD:D_SMA-SMB_Universal_Handsoldering -> Diode_SMD:D_SMA_Handsoldering
- R19, R20: footprint Resistor_SMD:R_1206_3216Metric_Pad1.42x1.75mm_HandSolder -> Resistor_SMD:R_0603_1608Metric_Pad1.05x0.95mm_HandSolder
- R3: footprint Resistor_SMD:R_0603_1608Metric_Pad1.05x0.95mm_HandSolder -> Resistor_SMD:R_1206_3216Metric_Pad1.42x1.75mm_HandSolder
- SW1: value RST -> PB
- SW3: value USR_BTN -> PB
- moved L1 141.2 mm to (60.6, 53.2), turned to 90 degrees
- moved C35 132.5 mm to (66.7, 118.4), turned to 270 degrees
- moved C34 129.3 mm to (68.7, 118.4), turned to 270 degrees
- moved C31 129.0 mm to (68.8, 108.3), turned to 90 degrees
- moved C33 127.6 mm to (63.0, 108.1), turned to 90 degrees
- moved C29 116.9 mm to (82.8, 118.4), turned to 270 degrees
- moved C28 105.2 mm to (85.3, 109.5), turned to 90 degrees
- moved U4 103.2 mm to (75.7, 113.3), turned to 180 degrees
- moved C30 96.1 mm to (83.1, 109.6), turned to 90 degrees
- moved C27 89.8 mm to (84.7, 118.5), turned to 270 degrees
- moved Y1 85.7 mm to (115.6, 102.3), turned to 180 degrees
- moved C11 85.2 mm to (118.6, 105.1), turned to 180 degrees
- moved C12 84.8 mm to (112.7, 105.1)
- moved R3 77.6 mm to (119.1, 97.9), turned to 270 degrees
- moved TP18 46.0 mm to (130.8, 83.8)
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Connections:
- C14 pad 1: /OSC32_IN -> GND
- C14 pad 2: GND -> /OSC32_IN
- C31 pad 2: /rs485/AUX_GND -> GNDD
- D7 pad 1: /RS485_A -> /RS485_B
- D7 pad 2: /RS485_B -> /RS485_A
- JP1 pad 1: /RS485_B -> /RS485_A
- R1 pad 2: Net-(J1-Pad3) -> GND
- R2 pad 1: Net-(J1-Pad4) -> GND
- R24 pad 2: /RS485_A -> /RS485_B
- U4 pad 11: /rs485/AUX_GND -> GNDD
Routing:
- net /RS485_A: track 8.77 -> 64.9 mm
- net /BOOT1: track 65.3 -> 12.9 mm
- net /DE~RE: track 89.3 -> 131.9 mm, vias 0 -> 1
- net /UART1_TX: track 118.8 -> 81.5 mm, vias 4 -> 0
- net +5V: track 139.4 -> 103.0 mm
- net /UART3_RX: track 157.8 -> 123.8 mm, vias 8 -> 2
- net /UART3_TX: track 160.7 -> 128.0 mm, vias 4 -> 2
- net +3V3: track 353.1 -> 382.0 mm
- net /UART1_RX: track 108.4 -> 79.6 mm, vias 2 -> 0
- net /USR_BTN: track 7.65 -> 34.3 mm
- net GNDD: track 1.98 -> 23.4 mm
- net /OSC_IN: track 1.09 -> 22.2 mm
- net /BOOT0: track 69.1 -> 48.6 mm
- net GND: track 110.6 -> 91.8 mm, vias 147 -> 154
- net /RS485_B: track 19.2 -> 36.9 mm
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Other:
- rule via_min_drill: 0.3 -> 0.25
- board text removed: "B1"
- board text removed: "CLK"
- board text removed: "IO"
- board text removed: "RX"
- board text removed: "TX"

Commit message: tmp: last bit of changes
Parts:
- added REF**: Fiducial_0.75mm_Mask1.5mm, Fiducial:Fiducial_0.75mm_Mask1.5mm, F.Cu at (40.6, 125.7)
- added REF**: Fiducial_0.75mm_Mask1.5mm, Fiducial:Fiducial_0.75mm_Mask1.5mm, F.Cu at (40.6, 38.1)
- added REF**: Fiducial_0.75mm_Mask1.5mm, Fiducial:Fiducial_0.75mm_Mask1.5mm, F.Cu at (135.9, 38.1)
- added REF**: Fiducial_0.75mm_Mask1.5mm, Fiducial:Fiducial_0.75mm_Mask1.5mm, F.Cu at (135.9, 125.7)
- added REF**: MountingHole_3.5mm, MountingHole:MountingHole_3.5mm, F.Cu at (132.6, 33.0)
- moved TP5 46.7 mm to (129.5, 119.4)
- moved TP4 42.1 mm to (123.2, 119.4)
- moved TP6 38.1 mm to (116.8, 119.4)
Routing:
- net /UART3_RX: track 123.8 -> 130.5 mm
- net /UART3_TX: track 128.0 -> 133.4 mm
- net +3V3: track 382.0 -> 383.6 mm
- net GND: track 91.8 -> 92.9 mm, vias 154 -> 213
- net /MODBUS_A7: track 143.8 -> 144.6 mm
- net /USR_BTN: track 34.3 -> 34.8 mm
- net /DE~RE: vias 1 -> 2
Other:
- board text added: "B0=1 <--> B0=0 BOOT MODE CONTROL"
- board text added: "BIT OFF <-> BIT ON ModBUS address"
- board text added: "CLK"
- board text added: "IO"
- board text added: "OFF <---> ON"
- board text added: "RX"
- board text added: "TX"
- board text removed: "B0"
